File: PCB/Rev 1/plate.kicad_pcb (KiCad board)
At the start: 2 copper layers, 354 x 121 mm, 126 parts, among them SW10 EC_SW, SW11 EC_SW, SW12 EC_SW, SW13 EC_SW, SW14 EC_SW, SW15 EC_SW, SW16 EC_SW, SW17 EC_SW, SW18 EC_SW, SW19 EC_SW, SW2 EC_SW, SW20 EC_SW, SW21 EC_SW, SW22 EC_SW, SW23 EC_SW, SW24 EC_SW, SW25 EC_SW, SW26 EC_SW, SW27 EC_SW, SW28 EC_SW, SW29 EC_SW, SW3 EC_SW, SW30 EC_SW, SW31 EC_SW, SW32 EC_SW, SW33 EC_SW, SW34 EC_SW, SW35 EC_SW, SW36 EC_SW, SW37 EC_SW, SW38 EC_SW, SW39 EC_SW, SW4 EC_SW, SW40 EC_SW, SW41 EC_SW, SW42 EC_SW, SW43 EC_SW, SW44 EC_SW, SW45 EC_SW, SW46 EC_SW, SW47 EC_SW, SW48 EC_SW, SW49 EC_SW, SW5 EC_SW, SW50 EC_SW, SW51 EC_SW, SW52 EC_SW, SW53 EC_SW, SW54 EC_SW, SW55 EC_SW, SW56 EC_SW, SW57 EC_SW, SW58 EC_SW, SW59 EC_SW, SW6 EC_SW, SW60 EC_SW, SW61 EC_SW, SW62 EC_SW, SW63 EC_SW, SW64 EC_SW, SW65 EC_SW, SW66 EC_SW, SW67 EC_SW, SW68 EC_SW, SW69 EC_SW, SW7 EC_SW, SW70 EC_SW, SW71 EC_SW, SW72 EC_SW, SW73 EC_SW, SW74 EC_SW, SW75 EC_SW, SW76 EC_SW, SW77 EC_SW, SW78 EC_SW, SW79 EC_SW, SW8 EC_SW, SW80 EC_SW, SW81 EC_SW, SW82 EC_SW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

Commit message: top mount plate addition and changed graphics
Parts:
- removed the G*** at (67.8, 105.3)
- added G***: LOGO, KeebGraphics:GhostrunnerSilk2, F.Cu at (365.3, 152.4)
- moved ? 11.2 mm to (342.5, 148.8)
- moved ? 11.2 mm to (210.8, 129.8)
- moved ? 11.2 mm to (358.2, 129.8)
- moved ? 11.2 mm to (316.6, 186.8)
- moved ? 11.2 mm to (225.1, 167.8)
- moved ? 11.2 mm to (358.2, 186.8)
- moved ? 11.2 mm to (244.1, 186.8)
- moved ? 11.2 mm to (139.6, 186.8)
- moved ? 11.2 mm to (291.6, 186.8)
- moved ? 11.2 mm to (378.3, 195.0)
- moved ? 11.2 mm to (267.8, 129.8)
- moved ? 11.2 mm to (130.1, 167.8)
- moved ? 11.2 mm to (367.7, 167.8)
- moved ? 11.2 mm to (134.8, 129.8)
- moved ? 11.2 mm to (274.7, 155.2)
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Routing:
- added copper zone on B.Cu, net (none)
- added copper zone on F.Cu, net (none)
Other:
- board size 354 x 121 mm -> 354 x 129 mm

Commit message: design changes
Parts:
- removed the ? at (378.3, 78.8)
- removed the ? at (29.1, 78.8)
- removed the ? at (29.1, 195.0)
- removed the ? at (378.3, 195.0)
- removed the G*** at (365.3, 152.4)
- added G***: LOGO, KeebGraphics:GhostrunnerSilk3, F.Cu at (364.5, 157.5)
Other:
- board size 354 x 129 mm -> 354 x 135 mm
